File: plus12/GridThumbs.brd (EAGLE design)
At the start: 114.3 x 21.6 mm, 14 parts

Commit message: Updates, BEFORE C5/6 Move
Routing:
- net N$6: track 135.5 -> 112.3 mm
- net N$14: track 30.4 -> 47.1 mm
- net N$3: track 73.9 -> 58.5 mm, vias 0 -> 2
- net N$5: track 103.1 -> 92.7 mm, vias 2 -> 4
- net N$21: track 49.4 -> 53.8 mm
- net N$19: track 131.0 -> 126.8 mm, vias 0 -> 1
- net N$4: track 103.0 -> 101.5 mm, vias 1 -> 3
- net N$2: track 53.9 -> 53.2 mm
