File: projects/plus12/CurvedThumbs.sch (EAGLE design)
At the start: 14 parts

Commit message: switching headers
Parts:
- removed INT2: INTRCNNT, Keys:INTRCNNT
- INT1: value INTRCNNT -> INTRCNNT4X2; device Keys:INTRCNNT -> Keys:INTRCNNT4X2
Connections:
- removed net N$14: INT1.T2, INT2.T1
- net N$10: no longer INT2.C4
- net N$11: no longer INT2.C5
- net N$12: no longer INT2.C6
- net N$7: no longer INT2.C1
- net N$8: no longer INT2.C2
- net N$9: no longer INT2.C3
Changed lines of the file:
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@@
 <?xml version="1.0" encoding="utf-8"?>
 <!DOCTYPE eagle SYSTEM "eagle.dtd">
-<eagle version="9.0.1">
+<eagle version="9.1.0">
 <drawing>
 <settings>
@@
 <part name="D5" library="Keys" library_urn="urn:adsk.eagle:library:1331239" deviceset="DIODE" device="" package3d_urn="urn:adsk.eagle:package:3624144/3"/>
 <part name="D6" library="Keys" library_urn="urn:adsk.eagle:library:1331239" deviceset="DIODE" device="" package3d_urn="urn:adsk.eagle:package:3624144/3"/>
-<part name="INT1" library="Keys" library_urn="urn:adsk.eagle:library:1331239" deviceset="INTRCNNT" device="" package3d_urn="urn:adsk.eagle:package:3650901/1"/>
-<part name="INT2" library="Keys" library_urn="urn:adsk.eagle:library:1331239" deviceset="INTRCNNT" device="" package3d_urn="urn:adsk.eagle:package:3650901/1"/>
+<part name="INT1" library="Keys" library_urn="urn:adsk.eagle:library:1331239" deviceset="INTRCNNT" device="4X2"/>
 </parts>
 <sheets>
@@
 <instance part="D6" gate="G$1" x="144.78" y="12.7" rot="R270"/>
 <instance part="INT1" gate="G$1" x="5.08" y="50.8" rot="R90"/>
-<instance part="INT2" gate="G$1" x="38.1" y="50.8" rot="R90"/>
 </instances>
 <busses>
@@
 <segment>
 <pinref part="INT1" gate="G$1" pin="C1"/>
-<wire x1="5.08" y1="50.8" x2="5.08" y2="48.26" width="0.1524" layer="91"/>
 <pinref part="SWI19" gate="G$1" pin="P1"/>
-<wire x1="5.08" y1="48.26" x2="5.08" y2="43.18" width="0.1524" layer="91"/>
+<wire x1="5.08" y1="50.8" x2="5.08" y2="43.18" width="0.1524" layer="91"/>
 <wire x1="5.08" y1="43.18" x2="0" y2="43.18" width="0.1524" layer="91"/>
 <wire x1="0" y1="43.18" x2="0" y2="25.4" width="0.1524" layer="91"/>
-<pinref part="INT2" gate="G$1" pin="C1"/>
-<wire x1="38.1" y1="50.8" x2="38.1" y2="48.26" width="0.1524" layer="91"/>
-<wire x1="38.1" y1="48.26" x2="5.08" y2="48.26" width="0.1524" layer="91"/>
-<junction x="5.08" y="48.26"/>
 </segment>
 </net>
@@
 <pinref part="INT1" gate="G$1" pin="C2"/>
 <wire x1="7.62" y1="50.8" x2="7.62" y2="33.02" width="0.1524" layer="91"/>
-<wire x1="7.62" y1="33.02" x2="22.86" y2="33.02" width="0.1524" layer="91"/>
+<wire x1="7.62" y1="33.02" x2="25.4" y2="33.02" width="0.1524" layer="91"/>
 <pinref part="SWI20" gate="G$1" pin="P1"/>
-<wire x1="22.86" y1="33.02" x2="25.4" y2="33.02" width="0.1524" layer="91"/>
 <wire x1="25.4" y1="33.02" x2="25.4" y2="25.4" width="0.1524" layer="91"/>
-<pinref part="INT2" gate="G$1" pin="C2"/>
-<wire x1="40.64" y1="50.8" x2="40.64" y2="45.72" width="0.1524" layer="91"/>
-<wire x1="40.64" y1="45.72" x2="22.86" y2="45.72" width="0.1524" layer="91"/>
-<wire x1="22.86" y1="45.72" x2="22.86" y2="33.02" width="0.1524" layer="91"/>
-<junction x="22.86" y="33.02"/>
 </segment>
 </net>
@@
 <wire x1="10.16" y1="50.8" x2="10.16" y2="35.56" width="0.1524" layer="91"/>
 <pinref part="SWI21" gate="G$1" pin="P1"/>
-<wire x1="10.16" y1="35.56" x2="43.18" y2="35.56" width="0.1524" layer="91"/>
-<wire x1="43.18" y1="35.56" x2="50.8" y2="35.56" width="0.1524" layer="91"/>
+<wire x1="10.16" y1="35.56" x2="50.8" y2="35.56" width="0.1524" layer="91"/>
 <wire x1="50.8" y1="35.56" x2="50.8" y2="25.4" width="0.1524" layer="91"/>
-<pinref part="INT2" gate="G$1" pin="C3"/>
-<wire x1="43.18" y1="50.8" x2="43.18" y2="35.56" width="0.1524" layer="91"/>
-<junction x="43.18" y="35.56"/>
 </segment>
 </net>
@@
 <pinref part="INT1" gate="G$1" pin="C4"/>
 <wire x1="12.7" y1="50.8" x2="12.7" y2="38.1" width="0.1524" layer="91"/>
-<wire x1="12.7" y1="38.1" x2="45.72" y2="38.1" width="0.1524" layer="91"/>
+<wire x1="12.7" y1="38.1" x2="76.2" y2="38.1" width="0.1524" layer="91"/>
 <pinref part="SWI22" gate="G$1" pin="P1"/>
-<wire x1="45.72" y1="38.1" x2="76.2" y2="38.1" width="0.1524" layer="91"/>
 <wire x1="76.2" y1="38.1" x2="76.2" y2="25.4" width="0.1524" layer="91"/>
-<pinref part="INT2" gate="G$1" pin="C4"/>
-<wire x1="45.72" y1="50.8" x2="45.72" y2="38.1" width="0.1524" layer="91"/>
-<junction x="45.72" y="38.1"/>
 </segment>
 </net>
@@
 <pinref part="INT1" gate="G$1" pin="C5"/>
 <wire x1="15.24" y1="50.8" x2="15.24" y2="40.64" width="0.1524" layer="91"/>
-<wire x1="15.24" y1="40.64" x2="48.26" y2="40.64" width="0.1524" layer="91"/>
 <pinref part="SWI23" gate="G$1" pin="P1"/>
-<wire x1="48.26" y1="40.64" x2="101.6" y2="40.64" width="0.1524" layer="91"/>
+<wire x1="15.24" y1="40.64" x2="101.6" y2="40.64" width="0.1524" layer="91"/>
 <wire x1="101.6" y1="40.64" x2="101.6" y2="25.4" width="0.1524" layer="91"/>
-<pinref part="INT2" gate="G$1" pin="C5"/>
-<wire x1="48.26" y1="50.8" x2="48.26" y2="40.64" width="0.1524" layer="91"/>
-<junction x="48.26" y="40.64"/>
 </segment>
 </net>
@@
 <wire x1="17.78" y1="50.8" x2="17.78" y2="43.18" width="0.1524" layer="91"/>
 <pinref part="SWI24" gate="G$1" pin="P1"/>
-<wire x1="17.78" y1="43.18" x2="50.8" y2="43.18" width="0.1524" layer="91"/>
-<wire x1="50.8" y1="43.18" x2="127" y2="43.18" width="0.1524" layer="91"/>
+<wire x1="17.78" y1="43.18" x2="127" y2="43.18" width="0.1524" layer="91"/>
 <wire x1="127" y1="43.18" x2="127" y2="25.4" width="0.1524" layer="91"/>
-<pinref part="INT2" gate="G$1" pin="C6"/>
-<wire x1="50.8" y1="50.8" x2="50.8" y2="43.18" width="0.1524" layer="91"/>
-<junction x="50.8" y="43.18"/>
 </segment>
 </net>
@@
 </segment>
 </net>
-<net name="N$14" class="0">
-<segment>
-<pinref part="INT1" gate="G$1" pin="T2"/>
-<wire x1="22.86" y1="50.8" x2="27.94" y2="50.8" width="0.1524" layer="91"/>
-<wire x1="27.94" y1="50.8" x2="27.94" y2="66.04" width="0.1524" layer="91"/>
-<wire x1="27.94" y1="66.04" x2="63.5" y2="66.04" width="0.1524" layer="91"/>
-<wire x1="63.5" y1="66.04" x2="63.5" y2="48.26" width="0.1524" layer="91"/>
-<wire x1="63.5" y1="48.26" x2="53.34" y2="48.26" width="0.1524" layer="91"/>
-<pinref part="INT2" gate="G$1" pin="T1"/>
-<wire x1="53.34" y1="48.26" x2="53.34" y2="50.8" width="0.1524" layer="91"/>
-</segment>
-</net>

Commit message: more updates than should be in one commit, lots of work
Changed lines of the file:
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@@
 <?xml version="1.0" encoding="utf-8"?>
 <!DOCTYPE eagle SYSTEM "eagle.dtd">
-<eagle version="9.1.0">
+<eagle version="9.1.1">
 <drawing>
 <settings>
