File: projects/plus12/GridThumbs.brd (EAGLE design)
At the start: 114.3 x 21.6 mm, 14 parts

Commit message: switching interconnects
Parts:
- removed INT2: INTRCNNT, Keys:INTRCNNT
- INT1: value INTRCNNT -> INTRCNNT4X2; device Keys:INTRCNNT -> Keys:INTRRIBBON
- moved INT1 30.7 mm to (40.6, 14.6)
- moved D20 19.1 mm to (34.3, 25.7)
- moved D19 19.1 mm to (15.2, 25.7)
- moved D21 19.1 mm to (53.3, 25.7)
- moved D22 12.8 mm to (72.4, 25.7), turned to 90 degrees
- moved D23 12.8 mm to (91.4, 25.7), turned to 90 degrees
- moved D24 12.8 mm to (110.5, 25.7), turned to 90 degrees
Connections:
- removed net N$14: INT1.T2, INT2.T1
- net N$19: now also INT1.T1
- net N$2: no longer INT2.C2
- net N$21: no longer INT1.T1, INT2.C1
- net N$3: no longer INT2.C3
- net N$4: no longer INT2.C4
- net N$5: no longer INT2.C5
- net N$6: no longer INT2.C6
Routing:
- net N$19: track 126.8 -> 0.00 mm, vias 1 -> 0
- net N$6: track 112.3 -> 0.00 mm
- net N$4: track 101.5 -> 0.00 mm, vias 3 -> 0
- net N$5: track 92.7 -> 0.00 mm, vias 4 -> 0
- net N$3: track 58.5 -> 0.00 mm, vias 2 -> 0
- net N$21: track 53.8 -> 0.00 mm
- net N$2: track 53.2 -> 0.00 mm, vias 1 -> 0
- net N$14: track 47.1 -> 0.00 mm
- net N$10: track 18.1 -> 0.00 mm
- net N$11: track 17.9 -> 0.00 mm
- net N$12: track 17.8 -> 0.00 mm
- net N$8: track 13.4 -> 0.00 mm
- net N$9: track 13.0 -> 0.00 mm
- net N$7: track 12.8 -> 0.00 mm
Other:
- board size 114.3 x 21.6 mm -> 116.2 x 25.4 mm
- board text added: "Panama Keynal"
- board text added: "Plus12"

Commit message: Getting ready for pictures
Parts:
- added U$1: (no value), Logos:3_8INCH_BOT
- added U$2: (no value), Logos:3_8INCH_TOP
Routing:
- net N$19: track 0.00 -> 144.3 mm
- net N$6: track 0.00 -> 84.9 mm
- net N$5: track 0.00 -> 68.5 mm
- net N$4: track 0.00 -> 40.7 mm
- net N$21: track 0.00 -> 32.4 mm
- net N$3: track 0.00 -> 26.2 mm
- net N$12: track 0.00 -> 21.4 mm
- net N$8: track 0.00 -> 21.4 mm
- net N$10: track 0.00 -> 21.4 mm
- net N$11: track 0.00 -> 20.9 mm
- net N$7: track 0.00 -> 20.9 mm
- net N$9: track 0.00 -> 20.9 mm
- net N$2: track 0.00 -> 20.0 mm

Commit message: more updates than should be in one commit, lots of work
Connections:
- net N$10: now also SWI22.RLMID
- net N$11: now also SWI23.RLMID
- net N$12: now also SWI24.RLMID
- net N$2: now also SWI20.LLP, SWI20.LRLP
- net N$21: now also SWI19.LLP, SWI19.LRLP
- net N$3: now also SWI21.LLP, SWI21.LRLP
- net N$4: now also SWI22.LLP, SWI22.LRLP
- net N$5: now also SWI23.LLP, SWI23.LRLP
- net N$6: now also SWI24.LLP, SWI24.LRLP
- net N$7: now also SWI19.RLMID
- net N$8: now also SWI20.RLMID
- net N$9: now also SWI21.RLMID
Routing:
- net N$7: track 20.9 -> 34.9 mm
- net N$9: track 20.9 -> 34.9 mm
- net N$11: track 20.9 -> 34.9 mm
- net N$12: track 21.4 -> 34.9 mm
- net N$8: track 21.4 -> 34.9 mm
- net N$10: track 21.4 -> 34.9 mm
- net N$5: track 68.5 -> 80.9 mm
- net N$6: track 84.9 -> 96.3 mm
- net N$4: track 40.7 -> 52.0 mm
- net N$3: track 26.2 -> 35.5 mm
- net N$2: track 20.0 -> 27.3 mm
- net N$19: track 144.3 -> 147.5 mm
- net N$21: track 32.4 -> 34.5 mm
Other:
- outline, holes or cut-outs redrawn
