File: projects/plus12/GridThumbs.sch (EAGLE design)
At the start: 14 parts

Commit message: switching interconnects
Parts:
- removed INT2: INTRCNNT, Keys:INTRCNNT
- INT1: value INTRCNNT -> INTRCNNT4X2; device Keys:INTRCNNT -> Keys:INTRCNNT4X2
Connections:
- removed net N$14: INT1.T2, INT2.T1
- net N$19: now also INT1.T1
- net N$2: no longer INT2.C2
- net N$21: no longer INT1.T1, INT2.C1
- net N$3: no longer INT2.C3
- net N$4: no longer INT2.C4
- net N$5: no longer INT2.C5
- net N$6: no longer INT2.C6
Changed lines of the file:
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@@
 <?xml version="1.0" encoding="utf-8"?>
 <!DOCTYPE eagle SYSTEM "eagle.dtd">
-<eagle version="9.0.1">
+<eagle version="9.1.0">
 <drawing>
 <settings>
@@
 <part name="D23" library="Keys" library_urn="urn:adsk.eagle:library:1331239" deviceset="DIODE" device="" package3d_urn="urn:adsk.eagle:package:3624144/3"/>
 <part name="D24" library="Keys" library_urn="urn:adsk.eagle:library:1331239" deviceset="DIODE" device="" package3d_urn="urn:adsk.eagle:package:3624144/3"/>
-<part name="INT1" library="Keys" library_urn="urn:adsk.eagle:library:1331239" deviceset="INTRCNNT" device="" package3d_urn="urn:adsk.eagle:package:3650901/1"/>
-<part name="INT2" library="Keys" library_urn="urn:adsk.eagle:library:1331239" deviceset="INTRCNNT" device="" package3d_urn="urn:adsk.eagle:package:3650901/1"/>
+<part name="INT1" library="Keys" library_urn="urn:adsk.eagle:library:1331239" deviceset="INTRCNNT" device="4X2"/>
 </parts>
 <sheets>
@@
 <instance part="D24" gate="G$1" x="144.78" y="38.1" rot="R270"/>
 <instance part="INT1" gate="G$1" x="0" y="76.2" rot="R90"/>
-<instance part="INT2" gate="G$1" x="35.56" y="76.2" rot="R90"/>
 </instances>
 <busses>
@@
 <wire x1="17.78" y1="55.88" x2="25.4" y2="55.88" width="0.1524" layer="91"/>
 <wire x1="25.4" y1="55.88" x2="25.4" y2="50.8" width="0.1524" layer="91"/>
-<pinref part="INT2" gate="G$1" pin="C2"/>
-<wire x1="38.1" y1="76.2" x2="38.1" y2="68.58" width="0.1524" layer="91"/>
-<wire x1="38.1" y1="68.58" x2="17.78" y2="68.58" width="0.1524" layer="91"/>
-<wire x1="17.78" y1="68.58" x2="17.78" y2="55.88" width="0.1524" layer="91"/>
-<junction x="17.78" y="55.88"/>
 </segment>
 </net>
@@
 <wire x1="40.64" y1="58.42" x2="50.8" y2="58.42" width="0.1524" layer="91"/>
 <wire x1="50.8" y1="58.42" x2="50.8" y2="50.8" width="0.1524" layer="91"/>
-<pinref part="INT2" gate="G$1" pin="C3"/>
-<wire x1="40.64" y1="76.2" x2="40.64" y2="58.42" width="0.1524" layer="91"/>
-<junction x="40.64" y="58.42"/>
 </segment>
 </net>
@@
 <wire x1="43.18" y1="60.96" x2="76.2" y2="60.96" width="0.1524" layer="91"/>
 <wire x1="76.2" y1="60.96" x2="76.2" y2="50.8" width="0.1524" layer="91"/>
-<pinref part="INT2" gate="G$1" pin="C4"/>
-<wire x1="43.18" y1="76.2" x2="43.18" y2="60.96" width="0.1524" layer="91"/>
-<junction x="43.18" y="60.96"/>
 </segment>
 </net>
@@
 <wire x1="45.72" y1="63.5" x2="101.6" y2="63.5" width="0.1524" layer="91"/>
 <wire x1="101.6" y1="63.5" x2="101.6" y2="50.8" width="0.1524" layer="91"/>
-<pinref part="INT2" gate="G$1" pin="C5"/>
-<wire x1="45.72" y1="76.2" x2="45.72" y2="63.5" width="0.1524" layer="91"/>
-<junction x="45.72" y="63.5"/>
 </segment>
 </net>
@@
 <wire x1="48.26" y1="66.04" x2="127" y2="66.04" width="0.1524" layer="91"/>
 <wire x1="127" y1="66.04" x2="127" y2="50.8" width="0.1524" layer="91"/>
-<pinref part="INT2" gate="G$1" pin="C6"/>
-<wire x1="48.26" y1="76.2" x2="48.26" y2="66.04" width="0.1524" layer="91"/>
-<junction x="48.26" y="66.04"/>
 </segment>
 </net>
@@
 <pinref part="D19" gate="G$1" pin="CAT"/>
 <pinref part="D20" gate="G$1" pin="CAT"/>
-<wire x1="17.78" y1="33.02" x2="43.18" y2="33.02" width="0.1524" layer="91"/>
+<wire x1="17.78" y1="33.02" x2="20.32" y2="33.02" width="0.1524" layer="91"/>
 <pinref part="D21" gate="G$1" pin="CAT"/>
+<wire x1="20.32" y1="33.02" x2="43.18" y2="33.02" width="0.1524" layer="91"/>
 <wire x1="43.18" y1="33.02" x2="68.58" y2="33.02" width="0.1524" layer="91"/>
 <junction x="43.18" y="33.02"/>
@@
 <wire x1="119.38" y1="33.02" x2="144.78" y2="33.02" width="0.1524" layer="91"/>
 <junction x="119.38" y="33.02"/>
+<pinref part="INT1" gate="G$1" pin="T1"/>
+<wire x1="15.24" y1="76.2" x2="15.24" y2="68.58" width="0.1524" layer="91"/>
+<wire x1="15.24" y1="68.58" x2="20.32" y2="68.58" width="0.1524" layer="91"/>
+<wire x1="20.32" y1="68.58" x2="20.32" y2="33.02" width="0.1524" layer="91"/>
+<junction x="20.32" y="33.02"/>
 </segment>
 </net>
@@
 <pinref part="INT1" gate="G$1" pin="C1"/>
 <wire x1="0" y1="76.2" x2="0" y2="71.12" width="0.1524" layer="91"/>
-<junction x="0" y="50.8"/>
-<pinref part="INT1" gate="G$1" pin="T1"/>
 <wire x1="0" y1="71.12" x2="0" y2="50.8" width="0.1524" layer="91"/>
-<wire x1="15.24" y1="76.2" x2="15.24" y2="68.58" width="0.1524" layer="91"/>
-<wire x1="15.24" y1="68.58" x2="-7.62" y2="68.58" width="0.1524" layer="91"/>
-<wire x1="-7.62" y1="68.58" x2="-7.62" y2="50.8" width="0.1524" layer="91"/>
-<wire x1="-7.62" y1="50.8" x2="0" y2="50.8" width="0.1524" layer="91"/>
-<pinref part="INT2" gate="G$1" pin="C1"/>
-<wire x1="35.56" y1="76.2" x2="35.56" y2="71.12" width="0.1524" layer="91"/>
-<wire x1="35.56" y1="71.12" x2="0" y2="71.12" width="0.1524" layer="91"/>
-<junction x="0" y="71.12"/>
-</segment>
-</net>
-<net name="N$14" class="0">
-<segment>
-<pinref part="INT2" gate="G$1" pin="T1"/>
-<wire x1="50.8" y1="76.2" x2="50.8" y2="73.66" width="0.1524" layer="91"/>
-<pinref part="INT1" gate="G$1" pin="T2"/>
-<wire x1="50.8" y1="73.66" x2="17.78" y2="73.66" width="0.1524" layer="91"/>
-<wire x1="17.78" y1="73.66" x2="17.78" y2="76.2" width="0.1524" layer="91"/>
-</segment>
-</net>
+</segment>
+</net>

Commit message: more updates than should be in one commit, lots of work
Changed lines of the file:
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@@
 <?xml version="1.0" encoding="utf-8"?>
 <!DOCTYPE eagle SYSTEM "eagle.dtd">
-<eagle version="9.1.0">
+<eagle version="9.1.1">
 <drawing>
 <settings>
