File: projects/plus12/DoubleThumbs.brd (EAGLE design)
At the start: 122.6 x 38.1 mm, 27 parts, among them SW28 MX/ALPSDOUBLESIDED

Commit message: more updates than should be in one commit, lots of work
Routing:
- net N$14: track 184.3 -> 162.1 mm, vias 0 -> 1
- net N$20: track 184.0 -> 173.0 mm
- net N$19: track 156.3 -> 147.4 mm
- net N$1: track 32.1 -> 35.1 mm
Other:
- outline, holes or cut-outs redrawn
