File: projects/plus12/StraightThumbs.brd (EAGLE design)
At the start: 118.7 x 54 mm, 14 parts

Commit message: switching interconnects
Parts:
- removed INT2: INTRCNNT, Keys:INTRCNNT
- INT1: value INTRCNNT -> INTRCNNT4X2; device Keys:INTRCNNT -> Keys:INTRRIBBON
- moved D6 19.0 mm to (98.4, 46.4)
- moved INT1 6.48 mm to (17.1, 39.4)
- moved D1 0.63 mm to (8.89, 5.71)
Connections:
- removed net N$14: INT1.T2, INT2.T1
- net N$10: no longer INT2.C4
- net N$11: no longer INT2.C5
- net N$12: no longer INT2.C6
- net N$7: no longer INT2.C1
- net N$8: no longer INT2.C2
- net N$9: no longer INT2.C3
Routing:
- net N$13: track 204.0 -> 0.00 mm, vias 2 -> 0
- net N$12: track 102.1 -> 0.00 mm
- net N$11: track 90.1 -> 0.00 mm
- net N$10: track 76.6 -> 0.00 mm
- net N$9: track 65.1 -> 0.00 mm, vias 1 -> 0
- net N$7: track 45.1 -> 0.00 mm
- net N$8: track 25.5 -> 0.00 mm
- net N$4: track 24.3 -> 0.00 mm
- net N$2: track 24.0 -> 0.00 mm
- net N$3: track 23.9 -> 0.00 mm
- net N$1: track 22.0 -> 0.00 mm
- net N$5: track 21.5 -> 0.00 mm
- net N$14: track 20.4 -> 0.00 mm
- net N$6: track 12.9 -> 0.00 mm
Other:
- board size 118.7 x 54 mm -> 116.8 x 54.6 mm
- board text added: "Baja Keylifornia"
- board text added: "Plus12"

Commit message: Getting ready for pictures
Parts:
- added U$1: (no value), Logos:3_8INCH_TOP
- added U$2: (no value), Logos:3_8INCH_BOT
Routing:
- net N$13: track 0.00 -> 195.1 mm
- net N$12: track 0.00 -> 91.2 mm
- net N$11: track 0.00 -> 75.0 mm
- net N$10: track 0.00 -> 50.5 mm
- net N$7: track 0.00 -> 33.5 mm
- net N$9: track 0.00 -> 28.7 mm
- net N$4: track 0.00 -> 24.5 mm
- net N$2: track 0.00 -> 23.2 mm
- net N$3: track 0.00 -> 22.4 mm
- net N$1: track 0.00 -> 22.2 mm
- net N$5: track 0.00 -> 21.3 mm
- net N$6: track 0.00 -> 20.2 mm
- net N$8: track 0.00 -> 14.5 mm

Commit message: more updates than should be in one commit, lots of work
Connections:
- net N$1: now also SWI19.RLMID
- net N$10: now also SWI22.LLP, SWI22.LRLP
- net N$11: now also SWI23.LLP, SWI23.LRLP
- net N$12: now also SWI24.LLP, SWI24.LRLP
- net N$2: now also SWI20.RLMID
- net N$3: now also SWI21.RLMID
- net N$4: now also SWI22.RLMID
- net N$5: now also SWI23.RLMID
- net N$6: now also SWI24.RLMID
- net N$7: now also SWI19.LLP, SWI19.LRLP
- net N$8: now also SWI20.LLP, SWI20.LRLP
- net N$9: now also SWI21.LLP, SWI21.LRLP
Routing:
- net N$12: track 91.2 -> 111.1 mm
- net N$10: track 50.5 -> 68.5 mm
- net N$9: track 28.7 -> 45.6 mm
- net N$11: track 75.0 -> 90.4 mm
- net N$8: track 14.5 -> 29.9 mm
- net N$13: track 195.1 -> 180.4 mm, vias 0 -> 1
- net N$6: track 20.2 -> 34.7 mm
- net N$1: track 22.2 -> 35.7 mm
- net N$5: track 21.3 -> 34.7 mm
- net N$7: track 33.5 -> 45.9 mm
- net N$3: track 22.4 -> 34.7 mm
- net N$2: track 23.2 -> 35.0 mm
- net N$4: track 24.5 -> 35.3 mm
Other:
- outline, holes or cut-outs redrawn

Commit message: more updates than should be in one commit, lots of work
Routing:
- net N$13: track 180.4 -> 175.6 mm, vias 1 -> 3
- net N$10: track 68.5 -> 66.1 mm
- net N$11: track 90.4 -> 92.1 mm
- net N$12: track 111.1 -> 109.6 mm
- net N$2: track 35.0 -> 36.4 mm
Other:
- board size 116.8 x 54.6 mm -> 116.6 x 54.5 mm
